File: Digital_OTA_Tremolo.kicad_pcb (KiCad board)
At the start: 2 copper layers, 1 part

Commit message: updates
Parts:
- moved REF** 17.4 mm to (159.1, 99.7)
Changed lines of the file:
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@@
     (uvia_drill 0.1)
   )
-  (module Hammond1590:1590BB locked (layer F.Cu)
-    (at 141.732 100.076)
+  (module Hammond1590:1590BB (layer F.Cu)
+    (at 159.131 99.695)
     (descr "Inside Lid Width and Inside Box Height - https://www.hammfg.com/files/parts/pdf/1590BB.pdf")
     (fp_text reference REF** (at 1.27 -56.134) (layer F.SilkS)
@@
       (effects (font (size 1 1) (thickness 0.15)))
     )
-    (fp_line (start 42.037 51.689) (end 42.037 -51.308) (layer Dwgs.User) (width 0.12))
-    (fp_line (start -42.037 51.689) (end -42.037 -51.308) (layer Dwgs.User) (width 0.12))
+    (fp_line (start 42.037 51.689) (end 42.037 -48.387) (layer Dwgs.User) (width 0.12))
+    (fp_line (start -42.037 51.689) (end -42.037 -48.387) (layer Dwgs.User) (width 0.12))
     (fp_line (start -42.037 51.689) (end 42.037 51.689) (layer Dwgs.User) (width 0.12))
-    (fp_line (start -42.037 -51.308) (end 42.037 -51.308) (layer Dwgs.User) (width 0.12))
+    (fp_line (start -42.037 -48.387) (end 42.037 -48.387) (layer Dwgs.User) (width 0.12))
   )
 )

Commit message: updated readme
Parts:
- removed REF**: 1590BB, Hammond1590:1590BB
- added C1: 10uF, Capacitor_SMD:C_0805_2012Metric_Pad1.15x1.40mm_HandSolder, F.Cu at (125.2, -144.1)
- added C2: 100nF, Capacitor_SMD:C_0805_2012Metric_Pad1.15x1.40mm_HandSolder, F.Cu at (129.1, -144.1)
- added C7: 100nF, Capacitor_SMD:C_0805_2012Metric_Pad1.15x1.40mm_HandSolder, F.Cu at (123.8, -10.1)
- added C8: 100nF, Capacitor_SMD:C_0805_2012Metric_Pad1.15x1.40mm_HandSolder, F.Cu at (141.4, -7.56)
- added D1: D_Schottky, Diode_SMD:D_SMA_Handsoldering, F.Cu at (114.7, -133.7)
- added D2: LED, LED_SMD:LED_1206_3216Metric_Pad1.42x1.75mm_HandSolder, F.Cu at (156.3, -136.7)
- added D3: LED, LED_SMD:LED_1206_3216Metric_Pad1.42x1.75mm_HandSolder, F.Cu at (149.9, -132.3)
- added D4: LED, LED_SMD:LED_1206_3216Metric_Pad1.42x1.75mm_HandSolder, F.Cu at (142.9, -122.6)
- added D5: LED, LED_SMD:LED_1206_3216Metric_Pad1.42x1.75mm_HandSolder, F.Cu at (119.8, -33.3)
- added D6: LED, LED_SMD:LED_1206_3216Metric_Pad1.42x1.75mm_HandSolder, F.Cu at (123.2, -33.3)
- added J1: NRJ6HM-1-PRE, NeutrikNRJ:NRJxHx, F.Cu at (187.1, 30.4)
- added J2: Barrel_Jack_Switch, Connector_BarrelJack:BarrelJack_Horizontal, F.Cu at (118.3, -124.1)
- added J3: Conn_01x04, Connector_Molex:Molex_KK-254_AE-6410-04A_1x04_P2.54mm_Vertical, F.Cu at (136.3, -27.4)
- added J4: NRJ6HM-1-PRE, NeutrikNRJ:NRJxHx, F.Cu at (74.7, 30.7)
- added R1: 10K, Resistor_SMD:R_0805_2012Metric_Pad1.15x1.40mm_HandSolder, F.Cu at (147.6, -96.9)
- added R10: 10K, Resistor_SMD:R_0805_2012Metric_Pad1.15x1.40mm_HandSolder, F.Cu at (124.5, 21.6)
- added R11: 10K, Resistor_SMD:R_0805_2012Metric_Pad1.15x1.40mm_HandSolder, F.Cu at (140.3, -28.0)
- added R12: 10K, Resistor_SMD:R_0805_2012Metric_Pad1.15x1.40mm_HandSolder, F.Cu at (139.8, 23.5)
- added R13: 10K, Resistor_SMD:R_0805_2012Metric_Pad1.15x1.40mm_HandSolder, F.Cu at (124.5, 23.5)
- added R14: 33K, Resistor_SMD:R_0805_2012Metric_Pad1.15x1.40mm_HandSolder, F.Cu at (139.8, 19.7)
- added R15: 33K, Resistor_SMD:R_0805_2012Metric_Pad1.15x1.40mm_HandSolder, F.Cu at (124.5, 19.7)
- added R16: 33K, Resistor_SMD:R_0805_2012Metric_Pad1.15x1.40mm_HandSolder, F.Cu at (139.8, 27.3)
- added R17: 33K, Resistor_SMD:R_0805_2012Metric_Pad1.15x1.40mm_HandSolder, F.Cu at (124.5, 27.3)
- added R18: 4K7, Resistor_SMD:R_0805_2012Metric_Pad1.15x1.40mm_HandSolder, F.Cu at (124.5, 29.2)
- added R19: 4K7, Resistor_SMD:R_0805_2012Metric_Pad1.15x1.40mm_HandSolder, F.Cu at (139.8, 29.2)
- added R2: 10K, Resistor_SMD:R_0805_2012Metric_Pad1.15x1.40mm_HandSolder, F.Cu at (142.6, -72.5)
- added R20: 1K, Resistor_SMD:R_0805_2012Metric_Pad1.15x1.40mm_HandSolder, F.Cu at (139.8, 31.1)
- added R21: 1K, Resistor_SMD:R_0805_2012Metric_Pad1.15x1.40mm_HandSolder, F.Cu at (124.5, 31.1)
- added R22: 2K7, Resistor_SMD:R_0805_2012Metric_Pad1.15x1.40mm_HandSolder, F.Cu at (141.4, -5.02)
- added R23: 2K7, Resistor_SMD:R_0805_2012Metric_Pad1.15x1.40mm_HandSolder, F.Cu at (141.4, -10.1)
- added R24: 1K, Resistor_SMD:R_0805_2012Metric_Pad1.15x1.40mm_HandSolder, F.Cu at (123.8, -6.29)
- added R25: 10K, Resistor_SMD:R_0805_2012Metric_Pad1.15x1.40mm_HandSolder, F.Cu at (123.8, -4.13)
- added R26: 10K, Resistor_SMD:R_0805_2012Metric_Pad1.15x1.40mm_HandSolder, F.Cu at (141.4, -12.1)
- added R27: 1K, Resistor_SMD:R_0805_2012Metric_Pad1.15x1.40mm_HandSolder, F.Cu at (162.0, -136.7)
- added R28: 1K, Resistor_SMD:R_0805_2012Metric_Pad1.15x1.40mm_HandSolder, F.Cu at (149.9, -126.6)
- added R29: 1K, Resistor_SMD:R_0805_2012Metric_Pad1.15x1.40mm_HandSolder, F.Cu at (137.2, -122.6)
- added R3: 10K, Resistor_SMD:R_0805_2012Metric_Pad1.15x1.40mm_HandSolder, F.Cu at (147.6, -72.5)
- added R30: 1K, Resistor_SMD:R_0805_2012Metric_Pad1.15x1.40mm_HandSolder, F.Cu at (119.8, -38.7)
- added R31: 1K, Resistor_SMD:R_0805_2012Metric_Pad1.15x1.40mm_HandSolder, F.Cu at (123.2, -38.7)
- added R4: 10k, Resistor_SMD:R_0805_2012Metric_Pad1.15x1.40mm_HandSolder, F.Cu at (123.8, -12.6)
- added R5: 10K, Resistor_SMD:R_0805_2012Metric_Pad1.15x1.40mm_HandSolder, F.Cu at (125.4, -97.8)
- added R6: 10K, Resistor_SMD:R_0805_2012Metric_Pad1.15x1.40mm_HandSolder, F.Cu at (118.4, -72.7)
- added R7: 4K7, Resistor_SMD:R_0805_2012Metric_Pad1.15x1.40mm_HandSolder, F.Cu at (123.8, -14.8)
- added R8: 10K, Resistor_SMD:R_0805_2012Metric_Pad1.15x1.40mm_HandSolder, F.Cu at (123.4, -72.6)
- added R9: 10K, Resistor_SMD:R_0805_2012Metric_Pad1.15x1.40mm_HandSolder, F.Cu at (139.8, 21.6)
- added RV1: B10K, Potentiometer_THT:Potentiometer_Bourns_PTV09A-1_Single_Vertical, F.Cu at (87.8, -46.9)
- added RV2: 1K, Potentiometer_SMD:Potentiometer_Bourns_3314J_Vertical, F.Cu at (132.1, 16.0)
- added SW1: Rotary_Encoder_Switch, Rotary_Encoder:RotaryEncoder_Alps_EC11E-Switch_Vertical_H20mm, F.Cu at (141.6, -78.8)
- added SW3: Rotary_Encoder_Switch, Rotary_Encoder:RotaryEncoder_Alps_EC11E-Switch_Vertical_H20mm, F.Cu at (119.4, -78.8)
- added SW_BYPASS1: SW_SPST, Connector_Molex:Molex_KK-254_AE-6410-02A_1x02_P2.54mm_Vertical, F.Cu at (149.1, -41.7)
- added SW_TAP1: SW_SPST, Connector_Molex:Molex_KK-254_AE-6410-02A_1x02_P2.54mm_Vertical, F.Cu at (149.1, -34.0)
- added U1: TL074, Package_SO:SOIC-16_3.9x9.9mm_P1.27mm, F.Cu at (132.7, -9.46)
- added U2: LM13700, Package_SO:SOIC-16_3.9x9.9mm_P1.27mm, F.Cu at (132.1, 24.1)
- added U3: STM32F072RBTx, Package_QFP:LQFP-64_10x10mm_P0.5mm, F.Cu at (132.5, -39.5)
- added U4: DG468DV_T1_E3, Package_TO_SOT_SMD:SOT-23-6_Handsoldering, F.Cu at (166.4, 35.5)
- added U5: RS6-0515D, RecomRS6:RS6, F.Cu at (134.2, -131.5)
- added U6: NCV5501_DT33RKG, Package_TO_SOT_SMD:TO-252-3_TabPin2, F.Cu at (139.8, -140.8)
- added U7: DG468DV_T1_E3, Package_TO_SOT_SMD:SOT-23-6_Handsoldering, F.Cu at (166.4, 23.7)
- added U8: DG468DV_T1_E3, Package_TO_SOT_SMD:SOT-23-6_Handsoldering, F.Cu at (93.0, 26.0)
Routing:
- net +3V3: track 0.00 -> 310.4 mm
- net VCOM: track 0.00 -> 186.7 mm, vias 0 -> 25
- net /SW_CLOSE_FX: track 0.00 -> 141.3 mm
- net Net-(U1-Pad3): track 0.00 -> 124.1 mm
- net Net-(J4-Pad1): track 0.00 -> 100.1 mm
- net /SINE1_TOGGLE_EXTI1: track 0.00 -> 75.1 mm
- net /SINE2_TOGGLE_EXTI2: track 0.00 -> 67.2 mm
- net Net-(R24-Pad2): track 0.00 -> 60.0 mm
- net /TIM2_CH2_ENCODER1: track 0.00 -> 58.3 mm
- net /TIM3_CH1_ENCODER2: track 0.00 -> 54.1 mm
- net +15V: track 0.00 -> 43.4 mm
- net /TIM2_CH1_ENCODER1: track 0.00 -> 38.9 mm
- net /TIM3_CH2_ENCODER2: track 0.00 -> 37.2 mm
- net Net-(C1-Pad1): track 0.00 -> 33.8 mm
- net /InvertInput: track 0.00 -> 26.6 mm
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